File: preamp-mar6.sch (KiCad schematic (older format))
At the start: 11 parts, among them J1 Pad, J2 Pad, J3 Pad, J4 Pad, U1 MAR6

Commit message: gg
Parts:
- C1, C2, C3: symbol xenir:Capacitor -> preamp-mar6-rescue:Capacitor-xenir
- C4: symbol xenir:Cap_Polarized -> preamp-mar6-rescue:Cap_Polarized-xenir
- J1, J2, J3, J4: symbol xenir:Pad -> preamp-mar6-rescue:Pad-xenir
- L1: value Inductor -> T37-43 10T; symbol xenir:Inductor -> preamp-mar6-rescue:Inductor-xenir
- R1: symbol xenir:Resistor -> preamp-mar6-rescue:Resistor-xenir
- U1: symbol xenir:MAR6 -> preamp-mar6-rescue:MAR6-xenir
Changed lines of the file:
@@
 $EndDescr
 $Comp
-L xenir:MAR6 U1
+L preamp-mar6-rescue:MAR6-xenir U1
 U 1 1 62D05110
 P 5650 4100
@@
 $EndComp
 $Comp
-L xenir:Inductor L1
+L preamp-mar6-rescue:Inductor-xenir L1
 U 1 1 62D06805
 P 6150 3800
 F 0 "L1" V 6104 3853 50  0000 L CNN
-F 1 "Inductor" V 6195 3853 50  0000 L CNN
+F 1 "T37-43 10T" V 6195 3853 50  0000 L CNN
 F 2 "xenir:T37_Inductor" H 6150 3900 50  0001 C CNN
 F 3 "" H 6150 3900 50  0001 C CNN
@@
 $EndComp
 $Comp
-L xenir:Resistor R1
+L preamp-mar6-rescue:Resistor-xenir R1
 U 1 1 62D0720F
 P 6150 3300
@@
 $EndComp
 $Comp
-L xenir:Capacitor C1
+L preamp-mar6-rescue:Capacitor-xenir C1
 U 1 1 62D07F71
 P 5000 4200
@@
 $EndComp
 $Comp
-L xenir:Capacitor C2
+L preamp-mar6-rescue:Capacitor-xenir C2
 U 1 1 62D0841D
 P 6550 4200
@@
 $EndComp
 $Comp
-L xenir:Capacitor C3
+L preamp-mar6-rescue:Capacitor-xenir C3
 U 1 1 62D08B85
 P 6700 3750
@@
 $EndComp
 $Comp
-L xenir:Cap_Polarized C4
+L preamp-mar6-rescue:Cap_Polarized-xenir C4
 U 1 1 62D09564
 P 7250 3750
@@
 $EndComp
 $Comp
-L xenir:Pad J3
+L preamp-mar6-rescue:Pad-xenir J3
 U 1 1 62D0A15C
 P 6000 2850
@@
 $EndComp
 $Comp
-L xenir:Pad J1
+L preamp-mar6-rescue:Pad-xenir J1
 U 1 1 62D0DBB4
 P 4550 4400
@@
 $EndComp
 $Comp
-L xenir:Pad J4
+L preamp-mar6-rescue:Pad-xenir J4
 U 1 1 62D0E480
 P 6700 4350
@@
 $EndComp
 $Comp
-L xenir:Pad J2
+L preamp-mar6-rescue:Pad-xenir J2
 U 1 1 62D0F60E
 P 5800 4700

Commit message: fixed - thanks Ali!
Connections:
- net +12V: now also C3.1, C4.1
- net at L1.1, R1.2: no longer C3.1, C4.1
Other:
- moved on the sheet: C3, C4
Changed lines of the file:
@@
 L preamp-mar6-rescue:Capacitor-xenir C3
 U 1 1 62D08B85
-P 6700 3750
-F 0 "C3" V 6671 3865 28  0000 L CNN
-F 1 ".1uF" V 6728 3865 28  0000 L CNN
-F 2 "xenir:Capacitor 1206" H 6700 3600 50  0001 C CNN
-F 3 "" H 6700 3600 50  0001 C CNN
-	1    6700 3750
+P 6700 3250
+F 0 "C3" V 6671 3365 28  0000 L CNN
+F 1 ".1uF" V 6728 3365 28  0000 L CNN
+F 2 "xenir:Capacitor 1206" H 6700 3100 50  0001 C CNN
+F 3 "" H 6700 3100 50  0001 C CNN
+	1    6700 3250
 	0    1    1    0
 $EndComp
@@
 L preamp-mar6-rescue:Cap_Polarized-xenir C4
 U 1 1 62D09564
-P 7250 3750
-F 0 "C4" V 7221 3768 28  0000 L CNN
-F 1 "10uF" V 7278 3768 28  0000 L CNN
-F 2 "xenir:Cap_4x5.4" H 7250 3800 50  0001 C CNN
-F 3 "" H 7250 3800 50  0001 C CNN
-	1    7250 3750
+P 7250 3250
+F 0 "C4" V 7221 3268 28  0000 L CNN
+F 1 "10uF" V 7278 3268 28  0000 L CNN
+F 2 "xenir:Cap_4x5.4" H 7250 3300 50  0001 C CNN
+F 3 "" H 7250 3300 50  0001 C CNN
+	1    7250 3250
 	0    1    1    0
 $EndComp
@@
 Connection ~ 6150 3000
 Wire Wire Line
-	6150 3500 6150 3600
-Wire Wire Line
-	6150 3600 6700 3600
-Connection ~ 6150 3600
-Wire Wire Line
-	6150 3600 6150 3650
-Wire Wire Line
-	6700 3600 7150 3600
-Connection ~ 6700 3600
+	6150 3100 6700 3100
+Wire Wire Line
+	6700 3100 7150 3100
+Connection ~ 6700 3100
 Wire Wire Line
 	6150 3950 6150 4200
@@
 L power:GND #PWR0104
 U 1 1 62D0C954
-P 6700 3900
-F 0 "#PWR0104" H 6700 3650 50  0001 C CNN
-F 1 "GND" H 6705 3727 50  0000 C CNN
-F 2 "" H 6700 3900 50  0001 C CNN
-F 3 "" H 6700 3900 50  0001 C CNN
-	1    6700 3900
+P 6700 3400
+F 0 "#PWR0104" H 6700 3150 50  0001 C CNN
+F 1 "GND" H 6705 3227 50  0000 C CNN
+F 2 "" H 6700 3400 50  0001 C CNN
+F 3 "" H 6700 3400 50  0001 C CNN
+	1    6700 3400
 	1    0    0    -1
 $EndComp
@@
 L power:GND #PWR0105
 U 1 1 62D0CCCC
-P 7150 3900
-F 0 "#PWR0105" H 7150 3650 50  0001 C CNN
-F 1 "GND" H 7155 3727 50  0000 C CNN
-F 2 "" H 7150 3900 50  0001 C CNN
-F 3 "" H 7150 3900 50  0001 C CNN
-	1    7150 3900
+P 7150 3400
+F 0 "#PWR0105" H 7150 3150 50  0001 C CNN
+F 1 "GND" H 7155 3227 50  0000 C CNN
+F 2 "" H 7150 3400 50  0001 C CNN
+F 3 "" H 7150 3400 50  0001 C CNN
+	1    7150 3400
 	1    0    0    -1
 $EndComp
@@
 EndData
 $EndBitmap
+Connection ~ 6150 3100
+Wire Wire Line
+	6150 3500 6150 3650
 $EndSCHEMATC
